File: 029/KiCad/esp32-programmer.sch (KiCad schematic (older format))
At the start: 33 parts, among them J1 USB_B, J2 Conn_02x03_Odd_Even, Q1 PUMX1, Q2 Q_PNP_BEC, Q3 Q_PNP_BEC, SW1 SW_Push_SPDT, U1 AMS1117-3.3, U2 CH340C

Commit message: updating partlist
Parts:
- Q1: value PUMX1 -> UMH3N
Changed lines of the file:
@@
 P 4250 3350
 F 0 "Q1" H 4441 3304 50  0000 L CNN
-F 1 "PUMX1" H 4441 3395 50  0000 L CNN
+F 1 "UMH3N" H 4441 3395 50  0000 L CNN
 F 2 "Package_TO_SOT_SMD:SOT-363_SC-70-6" H 4450 3450 50  0001 C CNN
 F 3 "https://assets.nexperia.com/documents/data-sheet/PUMX1.pdf" H 4250 3350 50  0001 C CNN
@@
 P 3650 3350
 F 0 "Q1" H 3841 3396 50  0000 L CNN
-F 1 "PUMX1" H 3841 3305 50  0000 L CNN
+F 1 "UMH3N" H 3841 3305 50  0000 L CNN
 F 2 "Package_TO_SOT_SMD:SOT-363_SC-70-6" H 3850 3450 50  0001 C CNN
 F 3 "https://assets.nexperia.com/documents/data-sheet/PUMX1.pdf" H 3650 3350 50  0001 C CNN
