File: 034/flipdot-brose-esp32.kicad_pcb (KiCad board)
At the start: 2 copper layers, 80 x 107 mm, 87 parts, among them J1 Conn_02x30_Odd_Even, J2 Barrel_Jack_Switch, J3 Screw_Terminal_01x02, J5 OLED, J6 TYPE-C-31-M-12, Q11 UMH3N, SW1 CONF, SW2 STAT, SW3 RST, U1 74HCT245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

Commit message: fixing naming SDA/SCL
Connections:
- J5 pad 3: SDA -> SCL
- J5 pad 4: SCL -> SDA
- R29 pad 1: SDA -> SCL
- R31 pad 2: SCL -> SDA
- U2 pad 8: SDA -> SCL
- U2 pad 9: SCL -> SDA
Routing:
- net SDA: track 48.4 -> 51.2 mm
- net SCL: track 51.2 -> 48.4 mm
